File: BMS_V2.kicad_pcb (KiCad board)
At the start: 2 copper layers, 156.7 x 80.6 mm, 143 parts, among them J1 BALANCING, J2 TEMP, J3 CAN OUT, J4 BATT_DCH, J6 BATT_IN, Q1 BSS84PWH6327XTSA1, Q10 BSS84PWH6327XTSA1, Q11 BSS84PWH6327XTSA1, Q12 BSS84PWH6327XTSA1, Q15 Q_NMOS_GDS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

Commit message: Add files via upload
Parts:
- Q15, Q18: value Q_NMOS_GDS -> 240N75F3
Connections:
- U8 pad 2: /BATTERY PROTECTION/DCH_SIG -> /BATTERY PROTECTION/CHG_SIG
- U8 pad 4: /BATTERY PROTECTION/CHG_SIG -> /BATTERY PROTECTION/DCH_SIG
Routing:
- net /BATTERY PROTECTION/DCH_SIG: track 194.1 -> 178.3 mm
- net /BATTERY PROTECTION/CHG_SIG: track 199.0 -> 194.5 mm
Changed lines of the file:
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@@
     (thickness 1.6)
     (drawings 7)
-    (tracks 1314)
+    (tracks 1313)
     (zones 0)
     (modules 143)
@@
       (effects (font (size 1 1) (thickness 0.15)))
     )
-    (fp_text value Q_NMOS_GDS (at 0 4.5 90) (layer F.Fab)
+    (fp_text value 240N75F3 (at 0 4.5 90) (layer F.Fab)
       (effects (font (size 1 1) (thickness 0.15)))
     )
@@
       (effects (font (size 1 1) (thickness 0.15)))
     )
-    (fp_text value Q_NMOS_GDS (at 0 4.5 270) (layer F.Fab)
+    (fp_text value 240N75F3 (at 0 4.5 270) (layer F.Fab)
       (effects (font (size 1 1) (thickness 0.15)))
     )
@@
       (net 120 "Net-(U8-Pad1)"))
     (pad 2 smd rect (at -2.7 -0.635) (size 1.55 0.6) (layers F.Cu F.Paste F.Mask)
-      (net 73 "/BATTERY PROTECTION/DCH_SIG"))
+      (net 72 "/BATTERY PROTECTION/CHG_SIG"))
     (pad 3 smd rect (at -2.7 0.635) (size 1.55 0.6) (layers F.Cu F.Paste F.Mask)
       (net 2 V-))
     (pad 4 smd rect (at -2.7 1.905) (size 1.55 0.6) (layers F.Cu F.Paste F.Mask)
-      (net 72 "/BATTERY PROTECTION/CHG_SIG"))
+      (net 73 "/BATTERY PROTECTION/DCH_SIG"))
     (pad 5 smd rect (at 2.7 1.905) (size 1.55 0.6) (layers F.Cu F.Paste F.Mask)
       (net 119 "Net-(Q18-Pad1)"))
@@
   (segment (start 183.0936 104.79) (end 184.14492 103.73868) (width 0.25) (layer F.Cu) (net 71))
   (segment (start 138.28014 78.37076) (end 138.2844 78.3665) (width 0.25) (layer F.Cu) (net 71))
-  (segment (start 195.58 82.677) (end 204.4446 82.677) (width 0.25) (layer B.Cu) (net 72))
-  (segment (start 90.7542 104.173) (end 89.2988 102.7176) (width 0.25) (layer F.Cu) (net 72))
-  (segment (start 90.7542 120.777) (end 90.7542 104.173) (width 0.25) (layer F.Cu) (net 72))
-  (segment (start 90.7796 120.8024) (end 90.7542 120.777) (width 0.25) (layer F.Cu) (net 72))
-  (via (at 90.7796 120.8024) (size 0.6) (drill 0.4) (layers F.Cu B.Cu) (net 72))
-  (segment (start 90.7796 127.0254) (end 90.7796 120.8024) (width 0.25) (layer B.Cu) (net 72))
-  (segment (start 94.615 130.8608) (end 90.7796 127.0254) (width 0.25) (layer B.Cu) (net 72))
-  (segment (start 201.9046 130.8608) (end 94.615 130.8608) (width 0.25) (layer B.Cu) (net 72))
-  (segment (start 208.3816 124.3838) (end 201.9046 130.8608) (width 0.25) (layer B.Cu) (net 72))
-  (segment (start 208.3816 86.614) (end 208.3816 124.3838) (width 0.25) (layer B.Cu) (net 72))
-  (segment (start 204.4446 82.677) (end 208.3816 86.614) (width 0.25) (layer B.Cu) (net 72))
-  (segment (start 89.2988 100.1776) (end 86.9188 100.1776) (width 0.25) (layer F.Cu) (net 73))
-  (segment (start 201.4728 85.217) (end 195.58 85.217) (width 0.25) (layer B.Cu) (net 73))
-  (segment (start 206.0194 89.7636) (end 201.4728 85.217) (width 0.25) (layer B.Cu) (net 73))
-  (segment (start 206.0194 123.5456) (end 206.0194 89.7636) (width 0.25) (layer B.Cu) (net 73))
-  (segment (start 200.7108 128.8542) (end 206.0194 123.5456) (width 0.25) (layer B.Cu) (net 73))
-  (segment (start 95.4278 128.8542) (end 200.7108 128.8542) (width 0.25) (layer B.Cu) (net 73))
-  (segment (start 95.0214 128.4478) (end 95.4278 128.8542) (width 0.25) (layer B.Cu) (net 73))
-  (via (at 95.0214 128.4478) (size 0.6) (drill 0.4) (layers F.Cu B.Cu) (net 73))
-  (segment (start 89.3572 122.7836) (end 95.0214 128.4478) (width 0.25) (layer F.Cu) (net 73))
-  (segment (start 89.3572 118.6942) (end 89.3572 122.7836) (width 0.25) (layer F.Cu) (net 73))
-  (segment (start 86.1822 115.5192) (end 89.3572 118.6942) (width 0.25) (layer F.Cu) (net 73))
-  (segment (start 86.1822 100.9142) (end 86.1822 115.5192) (width 0.25) (layer F.Cu) (net 73))
-  (segment (start 86.9188 100.1776) (end 86.1822 100.9142) (width 0.25) (layer F.Cu) (net 73))
+  (segment (start 195.58 82.677) (end 204.724 82.677) (width 0.25) (layer B.Cu) (net 72) (status 400000))
+  (segment (start 87.5792 100.1776) (end 89.2988 100.1776) (width 0.25) (layer F.Cu) (net 72) (status 800000))
+  (segment (start 87.0204 100.7364) (end 87.5792 100.1776) (width 0.25) (layer F.Cu) (net 72))
+  (segment (start 87.0204 105.0798) (end 87.0204 100.7364) (width 0.25) (layer F.Cu) (net 72))
+  (segment (start 88.4682 106.5276) (end 87.0204 105.0798) (width 0.25) (layer F.Cu) (net 72))
+  (segment (start 88.4682 118.0846) (end 88.4682 106.5276) (width 0.25) (layer F.Cu) (net 72))
+  (segment (start 91.1098 120.7262) (end 88.4682 118.0846) (width 0.25) (layer F.Cu) (net 72))
+  (via (at 91.1098 120.7262) (size 0.6) (drill 0.4) (layers F.Cu B.Cu) (net 72))
+  (segment (start 99.568 129.1844) (end 91.1098 120.7262) (width 0.25) (layer B.Cu) (net 72))
+  (segment (start 196.1134 129.1844) (end 99.568 129.1844) (width 0.25) (layer B.Cu) (net 72))
+  (segment (start 207.7974 117.5004) (end 196.1134 129.1844) (width 0.25) (layer B.Cu) (net 72))
+  (segment (start 207.7974 85.7504) (end 207.7974 117.5004) (width 0.25) (layer B.Cu) (net 72))
+  (segment (start 204.724 82.677) (end 207.7974 85.7504) (width 0.25) (layer B.Cu) (net 72))
+  (segment (start 89.2988 102.7176) (end 89.2988 116.4006) (width 0.25) (layer F.Cu) (net 73) (status 400000))
+  (segment (start 201.422 85.217) (end 195.58 85.217) (width 0.25) (layer B.Cu) (net 73) (status 800000))
+  (segment (start 205.2574 89.0524) (end 201.422 85.217) (width 0.25) (layer B.Cu) (net 73))
+  (segment (start 205.2574 117.729) (end 205.2574 89.0524) (width 0.25) (layer B.Cu) (net 73))
+  (segment (start 195.3514 127.635) (end 205.2574 117.729) (width 0.25) (layer B.Cu) (net 73))
+  (segment (start 104.14 127.635) (end 195.3514 127.635) (width 0.25) (layer B.Cu) (net 73))
+  (segment (start 103.9114 127.4064) (end 104.14 127.635) (width 0.25) (layer B.Cu) (net 73))
+  (via (at 103.9114 127.4064) (size 0.6) (drill 0.4) (layers F.Cu B.Cu) (net 73))
+  (segment (start 100.3046 127.4064) (end 103.9114 127.4064) (width 0.25) (layer F.Cu) (net 73))
+  (segment (start 89.2988 116.4006) (end 100.3046 127.4064) (width 0.25) (layer F.Cu) (net 73))
   (segment (start 177.59424 69.16928) (end 181.13756 69.16928) (width 0.25) (layer F.Cu) (net 74))
   (segment (start 181.13756 69.16928) (end 181.49316 69.52488) (width 0.25) (layer F.Cu) (net 74))
