File: bat_protection.sch (KiCad schematic (older format))
At the start: 7 parts, among them Q15 240N75F3, Q18 240N75F3, U7 ACS711xLCTR-25AB, U8 MIC4427

Commit message: Add files via upload
Connections:
- net CHG_SIG: now also U8.2 (IN_A); no longer U8.4 (IN_B)
- net DCH_SIG: now also U8.4 (IN_B); no longer U8.2 (IN_A)
Changed lines of the file:
@@
 	-1   0    0    1
 $EndComp
+Text HLabel 10200 3700 2    60   Input ~ 0
+CHG_SIG
 Text HLabel 10200 3500 2    60   Input ~ 0
-CHG_SIG
-Text HLabel 10200 3700 2    60   Input ~ 0
 DCH_SIG
 Text GLabel 4900 1800 0    60   Input ~ 0
